Commit message: added ros2 control

File: description/robot.urdf.xacro (robot description, xacro)
@@ -1,5 +1,13 @@
 <?xml version="1.0"?>
 <robot xmlns:xacro="http://www.ros.org/wiki/xacro"  name="robot">
+    <xacro:arg name="use_ros2_control" default="true"/>
     <xacro:include filename="robot_core.xacro" />
-    <xacro:include filename="gazebo_fourwheel_control.xacro"/>
+    <xacro:if value="$(arg use_ros2_control)">
+        <xacro:include filename="ros2_control.xacro"/>
+    </xacro:if>
+    <xacro:unless value="$(arg use_ros2_control)">
+        <xacro:include filename="gazebo_mod4.xacro"/>
+    </xacro:unless>
+    <!-- <xacro:include filename="gazebo_control.xacro"/> -->
+    <!-- <xacro:include filename="lidar.xacro"/> -->
 </robot>

File: description/robot_core.xacro (robot description, xacro)
@@ -13,4 +13,7 @@
     <material name="black">
         <color rgba="0 0 0 1"/>
+    </material>
+    <material name="red">
+        <color rgba="1 0 0 1"/>
     </material>
     <!-- BASE LINK -->
@@ -60,5 +63,5 @@
         <collision>
             <geometry>
-                <cylinder radius="0.05" length="0.04"/>
+                <sphere radius="0.05"/>
             </geometry>
         </collision>
@@ -86,5 +89,5 @@
         <collision>
             <geometry>
-                <cylinder radius="0.05" length="0.04"/>
+                <sphere radius="0.05"/>
             </geometry>
         </collision>
@@ -112,5 +115,5 @@
             <collision>
                 <geometry>
-                    <cylinder radius="0.05" length="0.04"/>
+                    <sphere radius="0.05"/>
                 </geometry>
             </collision>
@@ -138,5 +141,5 @@
             <collision>
                 <geometry>
-                    <cylinder radius="0.05" length="0.04"/>
+                    <sphere radius="0.05"/>
                 </geometry>
             </collision>
